File: KiCAD/USBaspProgrammer_Thomas-Fischl/USBaspProgrammer_Thomas-Fischl.kicad_sch (KiCad schematic)
At the start: 22 parts, among them J1 USB_B, J2 ISP_header_Conn_02x05_Odd_Even, U1 ATmega88-20PU, Y1 12MHz

Commit message: kicad
Parts:
- U1: footprint Package_DIP:DIP-28_W7.62mm -> My_Misc:DIP-28_W7.62mm_LongPads w socket
Changed lines of the file:
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@@
       (effects (font (size 1.27 1.27)) (justify right))
     )
-    (property "Footprint" "Package_DIP:DIP-28_W7.62mm" (id 2) (at 53.34 73.66 0)
+    (property "Footprint" "My_Misc:DIP-28_W7.62mm_LongPads w socket" (id 2) (at 53.34 73.66 0)
       (effects (font (size 1.27 1.27) italic) hide)
     )
@@
     )
     (path "/00000000-0000-0000-0000-000060289587"
-      (reference "U1") (unit 1) (value "ATmega88-20PU") (footprint "Package_DIP:DIP-28_W7.62mm")
+      (reference "U1") (unit 1) (value "ATmega88-20PU") (footprint "My_Misc:DIP-28_W7.62mm_LongPads w socket")
     )
     (path "/00000000-0000-0000-0000-000060292af4"
