File: KiCAD/devBoard/devBoard.kicad_sch (KiCad schematic)
At the start: 10 parts, among them J1 Conn_02x14_Counter_Clockwise, J2 ISP_header_Conn_02x05_Odd_Even, J3 ISP_header_Conn_02x05_Odd_Even, J4 ISP_header_Conn_02x05_Odd_Even, Y1 Crystal

Commit message: kicad
Parts:
- J1: renamed from J2; value ISP_header_Conn_02x05_Odd_Even -> ATmega88/328/328P
- J2: renamed from J3; value ISP_header_Conn_02x05_Odd_Even -> ATtiny4313
- J3: renamed from J4; value ISP_header_Conn_02x05_Odd_Even -> ATtiny85
- J4: renamed from J1; value Conn_02x14_Counter_Clockwise -> ZIF Socket
- JP1: value 3_pole_Jumper_2_Open -> ATmega88/328/328P
- JP2: value 3_pole_Jumper_2_Open -> ATtiny4313
- JP3: value 3_pole_Jumper_2_Open -> ATtiny85
- Y1: footprint My_Headers:3-pin_Crystal_header_large -> My_Headers:2-pin_Crystal_header_large
Connections:
- net 10: now also J2.8 (GND)
- net 4: now also J3.8 (GND)
- net 8: now also J1.8 (GND)
Other:
- note added: "Pin translation ___ 1 1 1 -| |- 8 20 28 2 2 2 -| |- 7 19 27 3 3 3 -| |- 6 18 26 4 4 4 -|___|- 5 17 25 5 5 -| |- 16 24 6 6 -| |- 15 23 7 7 -| |- 14 22 8 8 -| |- 13 21 9 9 -| |- 12 20 10 10 -|___|- 11 19 11 -| |- 18 12 -| |- 17 13 -| |- 16 14 -|___|- 15"
