File: KiCAD/devBoardv2/devBoardv2.kicad_sch (KiCad schematic)
At the start: 7 parts, among them J4 ISP header, U1 ATmega328-P, U2 ATtiny4313-P, U3 ATtiny85-20P, Y1 Crystal

Commit message: new kicad version
Parts:
- U1: footprint (none) -> My_Misc:ZIF_DIP_Socket-28_W6.9_W7.62_W7.62_W12.7_W13.5_w_dip_packet_large
- U2: footprint (none) -> My_Misc:ZIF_DIP_Socket-20_W4.3_W5.08_W7.62_W10.16_W10.9_3M_220-3342-00-0602J_w_dip_packet_large
- U3: footprint (none) -> My_Misc:DIP-8_W7.62mm_Socket_w_dip_packet_LongPads
