File: KiCAD/USBaspProgrammer-2in1/USBaspProgrammer-2in1.kicad_sch (KiCad schematic)
At the start: 22 parts, among them J1 USB_B, J2 ISP_header_Conn_02x05_Odd_Even, U1 ATmega88-20PU, Y1 12MHz

Commit message: schematics and pcb
Parts:
- added H1, H2, H3, H4: MountingHole, MountingHole:MountingHole_3.2mm_M3, symbol Mechanical:MountingHole
- added J7: ISP_header_Conn_02x03_Odd_Even, My_Misc:IDC-Header_2x03_P2.54mm_Horizontal_large, symbol My_Parts:ISP_header_Conn_02x03_Odd_Even
- D3: value LED green -> PWR
- D4: value LED red -> Progr
- JP1: renamed from JP2; value Self programming -> FW upg
- JP2: renamed from JP1; value Supply target -> PWR trgt
- JP3: value Slow SCK -> Slow CLK
Connections:
- net GND: now also J7.6 (GND)
- net at J2.5 (RST), JP1.2 (B), U1.16 (PB2): now also J7.5 (RST)
- net at J2.1 (MOSI), U1.17 (PB3): now also J7.4 (MOSI)
- net at J2.9 (MISO), U1.18 (PB4): now also J7.1 (MISO)
- net at J2.7 (SCK), U1.19 (PB5): now also J7.3 (SCK)
- net at J2.2 (VCC), JP2.2 (B): now also J7.2 (VCC)
Other:
- moved on the sheet: J2, R5
